Commit message: lx224hv stl file, common parameters and colors added

File: urdf/common/constants.xacro (robot description, xacro)
@@ -3,3 +3,4 @@
   <!-- Pi is already defined -->
   <!-- <xacro:property name="pi" value="3.14159265359"/> -->
+  <xacro:property name="scale" value="${1e-3}"/>
 </robot>

File: urdf/leg/leg.0.0.xacro (robot description, xacro)
@@ -5,5 +5,13 @@
   <xacro:property name="velocity" value="0.1"/>
   <xacro:macro name="leg" params="n xyz rpy parent">
-  <!-- Joint A1 or B1 -->
+  <!--
+  <joint name="leg${n}-servo-joint" type="fixed">
+    <parent link="${parent}"/>
+    <child link="leg${n}-servo1"/>
+    <origin rpy="0 0 0" xyz="0 0 0"/>
+  </joint>
+  <xacro:lx224 name="leg${n}-servo1" rpy="0 0 0" xyz="0 0 0" color="red"/>
+  -->
+  <!-- Leg Joint 1 -->
   <joint name="leg${n}_joint1" type="revolute">
     <parent link="${parent}"/>
@@ -18,12 +26,13 @@
         <box size="0.1 0.4 0.1"/>
       </geometry>
-      <origin xyz="0.0 0.2 0.0" rpy="0 0 0"/>
+      <origin xyz="0.0 0.4 0.0" rpy="0 0 0"/>
     </visual>
   </link>
+  <!-- Leg Joint 2 -->
   <joint name="leg${n}_joint2" type="revolute">
     <parent link="leg${n}_link1"/>
     <child link="leg${n}_link2"/>
     <origin xyz="0.0 0.6 0.0" rpy="0 0 0"/>
-    <axis xyz="1 0 0"/>
+    <axis xyz="0 0 1"/>
     <limit effort="100.0" velocity="1.0" lower="-${2*pi/3}" upper="${2*pi/3}"/>
   </joint>
@@ -33,13 +42,13 @@
         <box size="0.1 0.4 0.1"/>
       </geometry>
-      <origin xyz="0.0 0.2 0.0" rpy="0 0 0"/>
+      <origin xyz="0.0 0.4 0.0" rpy="0 0 0"/>
     </visual>
   </link>
-  <!-- Joint A3 or B3 -->
+  <!-- Leg Joint 3 -->
   <joint name="leg${n}_joint3" type="revolute">
     <parent link="leg${n}_link2"/>
     <child link="leg${n}_link3"/>
     <origin xyz="0.0 0.6 0.0" rpy="0 0 0"/>
-    <axis xyz="1 0 0"/>
+    <axis xyz="0 0 1"/>
     <limit effort="100.0" velocity="1.0" lower="-${2*pi/3}" upper="${2*pi/3}"/>
   </joint>
@@ -49,5 +58,5 @@
         <box size="0.1 0.4 0.1"/>
       </geometry>
-      <origin xyz="0.0 0.2 0.0" rpy="0 0 0"/>
+      <origin xyz="0.0 0.4 0.0" rpy="0 0 0"/>
     </visual>
   </link>

File: urdf/quaro.xacro (robot description, xacro)
@@ -1,6 +1,12 @@
 <?xml version="1.0"?>
 <robot name="quaro" xmlns:xacro="http://ros.org/wiki/xacro">
+  <!-- Various constant definitions -->
+  <xacro:include filename='$(find quaro_description)/urdf/common/constants.xacro'/>
+  <!-- Servo visual -->
+  <xacro:include filename="$(find quaro_description)/urdf/common/lx-224hv.xacro"/>
+  <!-- Material Colors -->
+  <xacro:include filename="$(find quaro_description)/urdf/common/colors.xacro"/>
+  <!-- Leg macro -->
   <xacro:include filename="$(find quaro_description)/urdf/leg/leg.0.0.xacro"/>
-  <xacro:include filename='$(find quaro_description)/urdf/common/constants.xacro'/>
   <!-- Base Link -->
   <link name="base_link">
@@ -13,6 +19,6 @@
   </link>
   <!-- Chain A -->
-  <xacro:leg n="1" parent="base_link" xyz="0.0 -0.2 0.0" rpy="${pi} 0 0"/>
+  <xacro:leg n="1" parent="base_link" xyz="0.0 -0.4 0.0" rpy="${pi} 0 ${pi/4}"/>
   <!-- Chain B -->
-  <xacro:leg n="2" parent="base_link" xyz="0.0 0.2 0.0" rpy="${pi} 0 -${pi}"/>
+  <xacro:leg n="2" parent="base_link" xyz="0.0 0.4 0.0" rpy="${pi} 0 ${3*pi/4}"/>
 </robot>
