Commit message: update urdf

File: urdf/leg/leg.0.0.xacro (robot description, xacro)
@@ -5,14 +5,13 @@
   <xacro:property name="velocity" value="0.1"/>
   <xacro:macro name="leg" params="n xyz rpy parent">
-  <!--
+<!--
   <joint name="leg${n}-servo-joint" type="fixed">
     <parent link="${parent}"/>
-    <child link="leg${n}-servo1"/>
+    <child link="hip_${n}"/>
     <origin rpy="0 0 0" xyz="0 0 0"/>
   </joint>
-  <xacro:lx224 name="leg${n}-servo1" rpy="0 0 0" xyz="0 0 0" color="red"/>
-  -->
+  <xacro:lx224 name="hip_${n}" rpy="0 0 0" xyz="0 0 0" color="red"/> -->
   <!-- Leg Joint 1 -->
-  <joint name="leg${n}_joint1" type="revolute">
+  <joint name="hip_${n}" type="revolute">
     <parent link="${parent}"/>
     <child link="leg${n}_link1"/>
@@ -30,8 +29,8 @@
   </link>
   <!-- Leg Joint 2 -->
-  <joint name="leg${n}_joint2" type="revolute">
+  <joint name="knee_${n}" type="revolute">
     <parent link="leg${n}_link1"/>
     <child link="leg${n}_link2"/>
-    <origin xyz="0.0 0.6 0.0" rpy="0 0 0"/>
+    <origin xyz="0.0 0.6 0.0" rpy="${pi/2} 0 0"/>
     <axis xyz="0 0 1"/>
     <limit effort="100.0" velocity="1.0" lower="-${2*pi/3}" upper="${2*pi/3}"/>
@@ -46,5 +45,5 @@
   </link>
   <!-- Leg Joint 3 -->
-  <joint name="leg${n}_joint3" type="revolute">
+  <joint name="ankle_${n}" type="revolute">
     <parent link="leg${n}_link2"/>
     <child link="leg${n}_link3"/>

File: urdf/quaro.xacro (robot description, xacro)
@@ -9,4 +9,6 @@
   <!-- Leg macro -->
   <xacro:include filename="$(find quaro_description)/urdf/leg/leg.0.0.xacro"/>
+  <!-- Import quaro ros2_control description -->
+  <xacro:include filename="$(find quaro_hardware_interface)/ros2_control/hardware_interface.ros2_control.xacro"/>
   <!-- Base Link -->
   <link name="base_link">
@@ -15,10 +17,15 @@
         <cylinder radius="0.1" length="0.2"/>
       </geometry>
-      <origin xyz="0 0 0" rpy="0 0 0"/>
+      <origin xyz="0 0 0" rpy="0 ${pi/2} 0"/>
     </visual>
   </link>
   <!-- Chain A -->
-  <xacro:leg n="1" parent="base_link" xyz="0.0 -0.4 0.0" rpy="${pi} 0 ${pi/4}"/>
+  <xacro:leg n="0" parent="base_link" xyz="0.1 -0.05 0.0" rpy="${pi} 0 ${pi/4}"/>
   <!-- Chain B -->
-  <xacro:leg n="2" parent="base_link" xyz="0.0 0.4 0.0" rpy="${pi} 0 ${3*pi/4}"/>
+  <xacro:leg n="1" parent="base_link" xyz="0.1 0.05 0.0" rpy="${pi} 0 ${3*pi/4}"/>
+  <!-- Chain B -->
+  <xacro:leg n="2" parent="base_link" xyz="-0.1 -0.05 0.0" rpy="${pi} 0 -${pi/4}"/>
+  <!-- Chain B -->
+  <xacro:leg n="3" parent="base_link" xyz="-0.1 0.05 0.0" rpy="${pi} 0 -${3*pi/4}"/>
+  <xacro:quaro_ros2_control/>
 </robot>

Commit message: meshes from the robot and urdf description

File: urdf/leg/leg.0.0.xacro (robot description, xacro)
@@ -4,12 +4,5 @@
   <xacro:property name="zero" value="0.0"/>
   <xacro:property name="velocity" value="0.1"/>
-  <xacro:macro name="leg" params="n xyz rpy parent">
-<!--
-  <joint name="leg${n}-servo-joint" type="fixed">
-    <parent link="${parent}"/>
-    <child link="hip_${n}"/>
-    <origin rpy="0 0 0" xyz="0 0 0"/>
-  </joint>
-  <xacro:lx224 name="hip_${n}" rpy="0 0 0" xyz="0 0 0" color="red"/> -->
+  <xacro:macro name="leg" params="n xyz rpy parent rot">
   <!-- Leg Joint 1 -->
   <joint name="hip_${n}" type="revolute">
@@ -17,5 +10,5 @@
     <child link="leg${n}_link1"/>
     <origin xyz="${xyz}" rpy="${rpy}"/>
-    <axis xyz="0 0 1"/>
+    <axis xyz="0 0 ${rot}"/>
     <limit effort="100.0" velocity="1.0" lower="-${2*pi/3}" upper="${2*pi/3}"/>
   </joint>
@@ -23,7 +16,7 @@
     <visual>
       <geometry>
-        <box size="0.1 0.4 0.1"/>
+        <mesh filename="package://quaro_description/meshes/hip_assembly.stl" scale="${scale} ${scale} ${scale}"/>
+      <origin xyz="0.0 0.0 0.0" rpy="0 0 0"/>
       </geometry>
-      <origin xyz="0.0 0.4 0.0" rpy="0 0 0"/>
     </visual>
   </link>
@@ -32,5 +25,5 @@
     <parent link="leg${n}_link1"/>
     <child link="leg${n}_link2"/>
-    <origin xyz="0.0 0.6 0.0" rpy="${pi/2} 0 0"/>
+    <origin xyz="${scale*40} ${scale*0} ${scale*28.3}" rpy="-${pi/2} 0 0"/>
     <axis xyz="0 0 1"/>
     <limit effort="100.0" velocity="1.0" lower="-${2*pi/3}" upper="${2*pi/3}"/>
@@ -39,7 +32,8 @@
     <visual>
       <geometry>
-        <box size="0.1 0.4 0.1"/>
+        <mesh filename="package://quaro_description/meshes/knee_assembly.stl" scale="${scale} ${scale} ${scale}"/>
       </geometry>
-      <origin xyz="0.0 0.4 0.0" rpy="0 0 0"/>
+      <origin xyz="${scale*10} ${scale*0} ${scale*0}" rpy="${pi/2} 0 ${pi}"/>
+      <material name="blue"/>
     </visual>
   </link>
@@ -48,5 +42,5 @@
     <parent link="leg${n}_link2"/>
     <child link="leg${n}_link3"/>
-    <origin xyz="0.0 0.6 0.0" rpy="0 0 0"/>
+    <origin xyz="${scale*53.9} ${scale*15} ${scale*0}" rpy="0 0 0"/>
     <axis xyz="0 0 1"/>
     <limit effort="100.0" velocity="1.0" lower="-${2*pi/3}" upper="${2*pi/3}"/>
@@ -55,7 +49,8 @@
     <visual>
       <geometry>
-        <box size="0.1 0.4 0.1"/>
+        <mesh filename="package://quaro_description/meshes/foot_assembly.stl" scale="${scale} ${scale} ${scale}"/>
       </geometry>
-      <origin xyz="0.0 0.4 0.0" rpy="0 0 0"/>
+      <origin xyz="${scale*10} ${scale*0} ${scale*0}" rpy="-${pi/2} 0 ${pi}"/>
+      <material name="green"/>
     </visual>
   </link>

File: urdf/quaro.xacro (robot description, xacro)
@@ -10,22 +10,23 @@
   <xacro:include filename="$(find quaro_description)/urdf/leg/leg.0.0.xacro"/>
   <!-- Import quaro ros2_control description -->
-  <xacro:include filename="$(find quaro_hardware_interface)/ros2_control/hardware_interface.ros2_control.xacro"/>
+  <!-- <xacro:include filename="$(find quaro_hardware_interface)/ros2_control/hardware_interface.ros2_control.xacro"/> -->
   <!-- Base Link -->
   <link name="base_link">
     <visual>
+      <origin xyz="0 0 0" rpy="${pi/2} 0 0"/>
       <geometry>
-        <cylinder radius="0.1" length="0.2"/>
+        <mesh filename="package://quaro_description/meshes/body_assembly.stl" scale="${scale} ${scale} ${scale}"/>
       </geometry>
-      <origin xyz="0 0 0" rpy="0 ${pi/2} 0"/>
+      <material name="gray"/>
     </visual>
   </link>
   <!-- Chain A -->
-  <xacro:leg n="0" parent="base_link" xyz="0.1 -0.05 0.0" rpy="${pi} 0 ${pi/4}"/>
+  <xacro:leg n="0" parent="base_link" rot="1" xyz="${scale*47} ${scale*91.5} ${scale*0.75}" rpy="0 0 ${pi/4}"/>
   <!-- Chain B -->
-  <xacro:leg n="1" parent="base_link" xyz="0.1 0.05 0.0" rpy="${pi} 0 ${3*pi/4}"/>
+  <xacro:leg n="1" parent="base_link" rot="-1" xyz="-${scale*47} ${scale*91.5} ${scale*0.75}" rpy="0 0 ${3*pi/4}"/>
   <!-- Chain B -->
-  <xacro:leg n="2" parent="base_link" xyz="-0.1 -0.05 0.0" rpy="${pi} 0 -${pi/4}"/>
+  <xacro:leg n="2" parent="base_link" rot="-1" xyz="${scale*47} -${scale*91.5} ${scale*0.75}" rpy="0 0 -${pi/4}"/>
   <!-- Chain B -->
-  <xacro:leg n="3" parent="base_link" xyz="-0.1 0.05 0.0" rpy="${pi} 0 -${3*pi/4}"/>
-  <xacro:quaro_ros2_control/>
+  <xacro:leg n="3" parent="base_link" rot="1" xyz="-${scale*47} -${scale*91.5} ${scale*0.75}" rpy="0 0 -${3*pi/4}"/>
+  <!-- <xacro:quaro_ros2_control/> -->
 </robot>
